Commit message: p3dx donusleri duzeltildi

File: xacro/p3dx/pioneer3dx_plugins.xacro (robot description, xacro)
@@ -22,6 +22,6 @@
             <rightJoint>right_hub_joint</rightJoint>
             <wheelSeparation>0.3</wheelSeparation>
-            <wheelDiameter>0.18</wheelDiameter>
-            <wheelTorque>20</wheelTorque>
+            <wheelDiameter>3.3</wheelDiameter>
+            <wheelTorque>25.0</wheelTorque>
             <wheelAcceleration>1.8</wheelAcceleration>
             <commandTopic>cmd_vel</commandTopic>

File: xacro/p3dx/pioneer3dx_wheel.xacro (robot description, xacro)
@@ -45,5 +45,5 @@
   <link name="${side}_wheel">
     <inertial>
-      <mass value="0.5"/>
+      <mass value="3.0"/>
       <origin xyz="0 0 0"/>
       <inertia ixx="0.012411765597" ixy="0" ixz="0" iyy="0.015218160428" iyz="0" izz="0.011763977943"/>
@@ -62,5 +62,5 @@
       <geometry>
         <!--<mesh filename="${meshes}/${side}_wheel.stl"/>-->
-        <cylinder radius="${radius}" length="0.01"/>
+        <cylinder radius="${radius}" length="15.0"/>
       </geometry>
     </collision>
