Commit message: gereksiz dosyalar silindi.

File: xacro/p3dx/pioneer3dx_chassis.xacro (robot description, xacro)
@@ -54,4 +54,27 @@
     <xacro:box_inertial x="0.445" y="0.38"  z="0.01" mass="1.0" />
   </link>
+<!-- gri kutu -->
+ <link name="simple_grey_box">
+    <inertial>
+      <mass value="0.01"/>
+      <origin xyz="0 0 0"/>
+      <inertia ixx="1" ixy="0" ixz="0" iyy="1" iyz="0" izz="1"/>
+    </inertial>
+    <visual name="base_visual">
+      <origin rpy="0 0 0" xyz="0 0 0"/>
+      <geometry name="top_geom">
+        <mesh filename="package://p3dx_description/meshes/top.stl"/>
+      </geometry>
+      <material name="TopBlack">
+        <color rgba="0.038 0.038 0.038 1.0"/>
+      </material>
+    </visual>
+    <collision>
+      <origin rpy="0 0 0" xyz="0.0 0 0"/>
+      <geometry name="pioneer_geom">
+        <box size="0.45 0.38 0.01"/>
+      </geometry>
+    </collision>
+  </link>
   <gazebo reference="top">
     <material value="Gazebo/Black"/>

Commit message: script dosyalarindaki hatalar duzeltildi. Calisir hale getirildi.

File: xacro/p3dx/pioneer3dx_chassis.xacro (robot description, xacro)
@@ -40,5 +40,5 @@
       <origin xyz="0 0 0" rpy="0 0 0"/>
       <geometry name="top_geom">
-        <mesh filename="${meshes}/top.stl"/>
+        <mesh filename="$(find quadro_demo)/person_standing/meshes/standing.dae"/>
       </geometry>
       <material name="TopBlack">
@@ -77,4 +77,16 @@
     </collision>
   </link>
+  <joint name="${name}_box_joint" type="fixed">
+    <origin xyz="-0.045 0 0.234" rpy="0 0 0"/>
+    <parent link="${name}"/>
+    <child link="box"/>
+  </joint>
+  <link name="box">
+        <visual>
+          <geometry>
+            <cylinder length="0.6" radius="0.2"/>
+          </geometry>
+        </visual>
+     </link>
   <gazebo reference="top">
     <material value="Gazebo/Black"/>
